Commit message: Fix position control and migrate teleop to ROS2

File: src/spot_mini_mini_description/urdf/ros2_control.xacro (robot description, xacro)
@@ -1,4 +1,4 @@
 <?xml version="1.0" ?>
-<<robot xmlns:xacro="http://www.ros.org/wiki/xacro">
+<robot xmlns:xacro="http://www.ros.org/wiki/xacro">
   <xacro:macro name="leg_ros2_control" params="leg">
     <joint name="motor_${leg}_hip">

File: src/spot_mini_mini_description/urdf/spot.urdf.xacro (robot description, xacro)
@@ -155,8 +155,8 @@
               i_rpy="0 0 0" i_xyz="-0.01 0 -0.06"
               mass="0.05"
-              c_xyz="0 0 -0.06"
-              length="0.035"
-              width="0.035"
-              height="0.12"
+              c_xyz="0 0 -0.04"
+              length="0.035"
+              width="0.035"
+              height="0.08"
               matname="black"
               meshfile="package://spot_mini_mini_description/meshes/OpenQuadruped/LEFT_LOWER_LEG.stl"
@@ -235,8 +235,8 @@
               i_rpy="0 0 0" i_xyz="-0.01 0 -0.06"
               mass="0.05"
-              c_xyz="0 0 -0.06"
-              length="0.035"
-              width="0.035"
-              height="0.12"
+              c_xyz="0 0 -0.04"
+              length="0.035"
+              width="0.035"
+              height="0.08"
               matname="black"
               meshfile="package://spot_mini_mini_description/meshes/OpenQuadruped/LEFT_LOWER_LEG.stl"
@@ -315,8 +315,8 @@
               i_rpy="0 0 0" i_xyz="-0.01 0 -0.06"
               mass="0.05"
-              c_xyz="0 0 -0.06"
-              length="0.035"
-              width="0.035"
-              height="0.12"
+              c_xyz="0 0 -0.04"
+              length="0.035"
+              width="0.035"
+              height="0.08"
               matname="black"
               meshfile="package://spot_mini_mini_description/meshes/OpenQuadruped/RIGHT_LOWER_LEG.stl"
@@ -395,8 +395,8 @@
               i_rpy="0 0 0" i_xyz="-0.01 0 -0.06"
               mass="0.05"
-              c_xyz="0 0 -0.06"
-              length="0.035"
-              width="0.035"
-              height="0.12"
+              c_xyz="0 0 -0.04"
+              length="0.035"
+              width="0.035"
+              height="0.08"
               matname="black"
               meshfile="package://spot_mini_mini_description/meshes/OpenQuadruped/RIGHT_LOWER_LEG.stl"

File: src/spot_mini_mini_description/urdf/spot_macro.xacro (robot description, xacro)
@@ -67,7 +67,9 @@
       </visual>
       <collision>
-        <origin rpy="${origin_rpy}" xyz="${c_xyz}" />
+        <!-- <origin rpy="${origin_rpy}" xyz="${c_xyz}" /> -->
+        <origin rpy="0 0 0" xyz="0 0 0" />
         <geometry>
-          <mesh filename="${meshfile}" scale="${meshscale}"/>
+          <!-- <mesh filename="${meshfile}" scale="${meshscale}"/> -->
+          <sphere radius="${radius}"/>
         </geometry>
         <contact_coefficients mu="10.1"/>
